File: GB2-KiCad/Control.kicad_sch (KiCad schematic)
At the start: 16 parts, among them Q10 2N7000, Q11 2N7000, Q12 2N7000, Q9 2N7000, U10 74LS14, U11 74LS08, U12 74LS02

Commit message: Added shunts and test points
Added shunt resistors and test points to the PCB for debugging purposes.
Parts:
- added C36, C37: 100nF, Capacitor_THT:C_Disc_D7.0mm_W2.5mm_P5.00mm, symbol Device:C
- added TP17, TP18, TP19, TP20, TP21, TP22, TP23, TP24, TP25, TP26, TP27, TP28: TestPoint, Connector_Pin:Pin_D1.0mm_L10.0mm, symbol Connector:TestPoint
Connections:
- net GNDD: now also C36.2, C37.2, TP23.1, TP24.1, TP25.1
- net Stage_1_Gate_1: now also TP17.1
- net Stage_1_Gate_2: now also TP18.1
- net VDD: now also C36.1, C37.1, TP26.1, TP27.1, TP28.1
- net at Q11.2 (G), U12.13: now also TP21.1
- net at Q10.2 (G), U11.6: now also TP20.1
- net at Q9.2 (G), U12.10: now also TP19.1
- net at Q12.2 (G), U11.8: now also TP22.1
