File: GB2-KiCad/GB2.kicad_pcb (KiCad board)
At the start: 2 copper layers, 41 parts, among them Q1 IRF540N, Q2 IRF540N, Q3 IRF540N, Q4 IRF540N, Q5 IPA60R180P7, Q6 IPA60R180P7, Q7 IPA60R180P7, Q8 IPA60R180P7, T1 Transformer_1P_1S, U1 IR2181, U2 IR2181, U3 TLP250, U4 TLP250, U5 TLP250, U6 TLP250

Commit message: Added shunts and test points
Added shunt resistors and test points to the PCB for debugging purposes.
Parts:
- added C10: 104, Capacitor_THT:C_Disc_D7.0mm_W2.5mm_P5.00mm, F.Cu at (437.0, 67.7)
- added C11: 50V 100uF, Capacitor_THT:CP_Radial_D10.0mm_P2.50mm_P5.00mm, F.Cu at (417.6, 42.9)
- added C12: 104, Capacitor_THT:C_Disc_D7.0mm_W2.5mm_P5.00mm, F.Cu at (437.0, 71.7)
- added C13: 50V 100uF, Capacitor_THT:CP_Radial_D10.0mm_P2.50mm_P5.00mm, F.Cu at (417.6, 54.4)
- added C14: 104, Capacitor_THT:C_Disc_D7.0mm_W2.5mm_P5.00mm, F.Cu at (437.0, 75.8)
- added C15: 50V 4700uF, Capacitor_THT:CP_Radial_D16.0mm_P7.50mm, F.Cu at (342.0, 61.4)
- added C16: 470V 220uF, Capacitor_THT:CP_Radial_D22.0mm_P10.00mm_SnapIn, F.Cu at (281.9, 110.7)
- added C17: 630VAC 0.24uF, Capacitor_THT:C_Rect_L33.0mm_W15.0mm_P27.50mm_MKS4, F.Cu at (127.0, 75.2)
- added C19: 50V 22uF, Capacitor_THT:CP_Radial_D5.0mm_P2.00mm, F.Cu at (460.8, 28.8)
- added C20: 50V 22uF, Capacitor_THT:CP_Radial_D5.0mm_P2.00mm, F.Cu at (460.8, 35.4)
- added C21: 50V 22uF, Capacitor_THT:CP_Radial_D5.0mm_P2.00mm, F.Cu at (460.8, 41.9)
- added C22: C_Polarized, Capacitor_THT:CP_Radial_D10.0mm_P2.50mm_P5.00mm, F.Cu at (369.6, 30.5)
- added C23: C_Polarized, Capacitor_THT:CP_Radial_D10.0mm_P2.50mm_P5.00mm, F.Cu at (369.6, 42.0)
- added C24: 5-65pF, GB2:C_Trim, F.Cu at (35.6, 35.6)
- added C25: 5-65pF, GB2:C_Trim, F.Cu at (45.7, 50.8)
- added C26: 5-65pF, GB2:C_Trim, F.Cu at (71.1, 33.0)
- added C27: C_Polarized, Capacitor_THT:CP_Radial_D10.0mm_P2.50mm_P5.00mm, F.Cu at (369.6, 53.6)
- added C28: 30pF, Capacitor_THT:C_Disc_D3.4mm_W2.1mm_P2.50mm, F.Cu at (171.4, 24.1)
- added C29: 30pF, Capacitor_THT:C_Disc_D3.4mm_W2.1mm_P2.50mm, F.Cu at (171.4, 49.5)
- added C30: 30pF, Capacitor_THT:C_Disc_D3.4mm_W2.1mm_P2.50mm, F.Cu at (414.4, 69.3)
- added C31: 30pF, Capacitor_THT:C_Disc_D3.4mm_W2.1mm_P2.50mm, F.Cu at (414.4, 73.0)
- added C32: 100nF, Capacitor_THT:C_Disc_D7.0mm_W2.5mm_P5.00mm, F.Cu at (55.9, 20.3)
- added C33: 100nF, Capacitor_THT:C_Disc_D7.0mm_W2.5mm_P5.00mm, F.Cu at (109.1, 22.9)
- added C34: 100nF, Capacitor_THT:C_Disc_D7.0mm_W2.5mm_P5.00mm, F.Cu at (121.8, 22.9)
- added C35: C_Polarized, Capacitor_THT:CP_Radial_D10.0mm_P2.50mm_P5.00mm, F.Cu at (369.6, 65.1)
- added C36: 100nF, Capacitor_THT:C_Disc_D7.0mm_W2.5mm_P5.00mm, F.Cu at (147.3, 39.8)
- added C37: 100nF, Capacitor_THT:C_Disc_D7.0mm_W2.5mm_P5.00mm, F.Cu at (147.3, 43.9)
- added C38: 400VDC 3.3uF, Capacitor_THT:C_Rect_L33.0mm_W15.0mm_P27.50mm_MKS4, F.Cu at (256.5, 129.5)
- added C5: 104, Capacitor_THT:C_Disc_D7.0mm_W2.5mm_P5.00mm, F.Cu at (188.0, 17.9)
- added C6: 104, Capacitor_THT:C_Disc_D7.0mm_W2.5mm_P5.00mm, F.Cu at (188.0, 43.3)
- added C7: 104, Capacitor_THT:C_Disc_D7.0mm_W2.5mm_P5.00mm, F.Cu at (188.0, -7.54)
- added C8: 104, Capacitor_THT:C_Disc_D7.0mm_W2.5mm_P5.00mm, F.Cu at (188.0, 68.7)
- added C9: 50V 100uF, Capacitor_THT:CP_Radial_D10.0mm_P2.50mm_P5.00mm, F.Cu at (157.2, 59.1)
- added D10: D_Zener, Diode_THT:D_DO-41_SOD81_P10.16mm_Horizontal, F.Cu at (457.2, 64.3)
- added D11: D_Zener, Diode_THT:D_DO-41_SOD81_P10.16mm_Horizontal, F.Cu at (457.2, 68.6)
- added D7: D_Zener, Diode_THT:D_DO-41_SOD81_P10.16mm_Horizontal, F.Cu at (457.2, 51.6)
- added D8: D_Zener, Diode_THT:D_DO-41_SOD81_P10.16mm_Horizontal, F.Cu at (457.2, 55.8)
- added D9: D_Zener, Diode_THT:D_DO-41_SOD81_P10.16mm_Horizontal, F.Cu at (457.2, 60.1)
- added J1: Screw_Terminal_01x02, TerminalBlock_Dinkle:TerminalBlock_Dinkle_DT-55-B01X-02_P10.00mm, F.Cu at (40.6, 190.3)
- added J2: Screw_Terminal_01x02, TerminalBlock_Dinkle:TerminalBlock_Dinkle_DT-55-B01X-02_P10.00mm, F.Cu at (381.0, 98.0)
- added J3: Barrel_Jack_Switch, Connector_BarrelJack:BarrelJack_GCT_DCJ200-10-A_Horizontal, F.Cu at (47.0, 165.1)
- added J4: Conn_02x10_Odd_Even, Connector_PinHeader_2.54mm:PinHeader_2x10_P2.54mm_Vertical, F.Cu at (22.9, 20.3)
- added L1: 42uH, Inductor_THT:L_Toroid_Vertical_L21.6mm_W8.4mm_P8.38mm_Pulse_G, F.Cu at (99.9, 86.4)
- added L2: L_Ferrite, Inductor_THT:L_Toroid_Vertical_L21.6mm_W8.4mm_P8.38mm_Pulse_G, F.Cu at (252.3, 83.8)
- added L3: 1000uH, Inductor_THT:L_Toroid_Vertical_L21.6mm_W8.4mm_P8.38mm_Pulse_G, F.Cu at (357.3, 97.8)
- added NT1: NetTie_2, NetTie:NetTie-2_SMD_Pad2.0mm, F.Cu at (43.2, 68.6)
- added PS1: ITX2412SA-HR, Converter_DCDC:Converter_DCDC_XP_POWER-ITxxxxxS_THT, F.Cu at (170.2, 55.9)
- added PS2: ITX2412SA-HR, Converter_DCDC:Converter_DCDC_XP_POWER-ITxxxxxS_THT, F.Cu at (170.2, 30.5)
- added PS3: ITX2412SA-HR, Converter_DCDC:Converter_DCDC_XP_POWER-ITxxxxxS_THT, F.Cu at (170.2, 5.08)
- added Q10: 2N7000, Package_TO_SOT_THT:TO-92L_HandSolder, F.Cu at (141.0, 35.3)
- added Q11: 2N7000, Package_TO_SOT_THT:TO-92L_HandSolder, F.Cu at (141.0, 41.4)
- added Q12: 2N7000, Package_TO_SOT_THT:TO-92L_HandSolder, F.Cu at (157.5, 68.6)
- added Q9: 2N7000, Package_TO_SOT_THT:TO-92L_HandSolder, F.Cu at (141.0, 29.2)
- added R10: R, Resistor_THT:R_Axial_DIN0204_L3.6mm_D1.6mm_P7.62mm_Horizontal, F.Cu at (426.1, 66.8)
- added R11: R, Resistor_THT:R_Axial_DIN0204_L3.6mm_D1.6mm_P7.62mm_Horizontal, F.Cu at (397.1, 78.9)
- added R12: R, Resistor_THT:R_Axial_DIN0204_L3.6mm_D1.6mm_P7.62mm_Horizontal, F.Cu at (426.1, 69.9)
- added R13: R, Resistor_THT:R_Axial_DIN0204_L3.6mm_D1.6mm_P7.62mm_Horizontal, F.Cu at (426.1, 73.1)
- added R14: R, Resistor_THT:R_Axial_DIN0204_L3.6mm_D1.6mm_P7.62mm_Horizontal, F.Cu at (426.1, 76.2)
- added R15: R, Resistor_THT:R_Axial_DIN0204_L3.6mm_D1.6mm_P7.62mm_Horizontal, F.Cu at (426.1, 79.4)
- added R16: 100k, Resistor_THT:R_Axial_DIN0204_L3.6mm_D1.6mm_P7.62mm_Horizontal, F.Cu at (43.2, 22.9)
- added R17: 100k, Resistor_THT:R_Axial_DIN0204_L3.6mm_D1.6mm_P7.62mm_Horizontal, F.Cu at (61.0, 45.7)
- added R18: 100k, Resistor_THT:R_Axial_DIN0204_L3.6mm_D1.6mm_P7.62mm_Horizontal, F.Cu at (155.5, 33.5)
- added R19: R, Resistor_THT:R_Axial_DIN0204_L3.6mm_D1.6mm_P7.62mm_Horizontal, F.Cu at (61.0, 182.9)
- added R20: R, Resistor_THT:R_Axial_DIN0204_L3.6mm_D1.6mm_P7.62mm_Horizontal, F.Cu at (48.3, 104.1)
- added R21: R, Resistor_THT:R_Axial_DIN0204_L3.6mm_D1.6mm_P7.62mm_Horizontal, F.Cu at (48.3, 144.8)
- added R22: R_Shunt, Resistor_THT:R_Axial_Shunt_L22.2mm_W8.0mm_PS14.30mm_P25.40mm, F.Cu at (129.5, 139.7)
- added R23: R_Shunt, Resistor_THT:R_Axial_Shunt_L22.2mm_W8.0mm_PS14.30mm_P25.40mm, F.Cu at (295.9, 91.4)
- added R24: R_Shunt, Resistor_THT:R_Axial_Shunt_L22.2mm_W8.0mm_PS14.30mm_P25.40mm, F.Cu at (408.9, 111.8)
- added R25: R_Shunt, Resistor_THT:R_Axial_Shunt_L22.2mm_W8.0mm_PS14.30mm_P25.40mm, F.Cu at (73.7, 165.1)
- added R9: R, Resistor_THT:R_Axial_DIN0204_L3.6mm_D1.6mm_P7.62mm_Horizontal, F.Cu at (426.1, 63.6)
- added TP1: TestPoint, Connector_Pin:Pin_D1.0mm_L10.0mm, F.Cu at (58.4, 204.2)
- added TP10: TestPoint, Connector_Pin:Pin_D1.0mm_L10.0mm, F.Cu at (152.4, 205.3)
- added TP11: TestPoint, Connector_Pin:Pin_D1.0mm_L10.0mm, F.Cu at (152.4, 209.3)
- added TP12: TestPoint, Connector_Pin:Pin_D1.0mm_L10.0mm, F.Cu at (152.4, 213.4)
- added TP13: TestPoint, Connector_Pin:Pin_D1.0mm_L10.0mm, F.Cu at (134.2, 205.3)
- added TP14: TestPoint, Connector_Pin:Pin_D1.0mm_L10.0mm, F.Cu at (134.2, 209.3)
- added TP15: TestPoint, Connector_Pin:Pin_D1.0mm_L10.0mm, F.Cu at (134.2, 213.4)
- added TP16: TestPoint, Connector_Pin:Pin_D1.0mm_L10.0mm, F.Cu at (134.2, 217.4)
- added TP17: TestPoint, Connector_Pin:Pin_D1.0mm_L10.0mm, F.Cu at (148.3, 183.0)
- added TP18: TestPoint, Connector_Pin:Pin_D1.0mm_L10.0mm, F.Cu at (148.3, 187.1)
- added TP19: TestPoint, Connector_Pin:Pin_D1.0mm_L10.0mm, F.Cu at (148.3, 191.1)
- added TP2: TestPoint, Connector_Pin:Pin_D1.0mm_L10.0mm, F.Cu at (58.4, 208.3)
- added TP20: TestPoint, Connector_Pin:Pin_D1.0mm_L10.0mm, F.Cu at (152.4, 183.0)
- added TP21: TestPoint, Connector_Pin:Pin_D1.0mm_L10.0mm, F.Cu at (152.4, 187.1)
- added TP22: TestPoint, Connector_Pin:Pin_D1.0mm_L10.0mm, F.Cu at (152.4, 191.1)
- added TP23: TestPoint, Connector_Pin:Pin_D1.0mm_L10.0mm, F.Cu at (156.4, 183.0)
- added TP24: TestPoint, Connector_Pin:Pin_D1.0mm_L10.0mm, F.Cu at (156.4, 187.1)
- added TP25: TestPoint, Connector_Pin:Pin_D1.0mm_L10.0mm, F.Cu at (156.4, 191.1)
- added TP26: TestPoint, Connector_Pin:Pin_D1.0mm_L10.0mm, F.Cu at (160.5, 183.0)
- added TP27: TestPoint, Connector_Pin:Pin_D1.0mm_L10.0mm, F.Cu at (160.5, 187.1)
- added TP28: TestPoint, Connector_Pin:Pin_D1.0mm_L10.0mm, F.Cu at (160.5, 191.1)
- added TP29: TestPoint, Connector_Pin:Pin_D1.0mm_L10.0mm, F.Cu at (134.2, 183.0)
- added TP3: TestPoint, Connector_Pin:Pin_D1.0mm_L10.0mm, F.Cu at (148.3, 197.2)
- added TP30: TestPoint, Connector_Pin:Pin_D1.0mm_L10.0mm, F.Cu at (134.2, 187.1)
- added TP31: TestPoint, Connector_Pin:Pin_D1.0mm_L10.0mm, F.Cu at (134.2, 191.1)
- added TP32: TestPoint, Connector_Pin:Pin_D1.0mm_L10.0mm, F.Cu at (134.2, 195.2)
- added TP33: TestPoint, Connector_Pin:Pin_D1.0mm_L10.0mm, F.Cu at (134.2, 199.2)
- added TP34: TestPoint, Connector_Pin:Pin_D1.0mm_L10.0mm, F.Cu at (138.2, 183.0)
- added TP35: TestPoint, Connector_Pin:Pin_D1.0mm_L10.0mm, F.Cu at (138.2, 187.1)
- added TP36: TestPoint, Connector_Pin:Pin_D1.0mm_L10.0mm, F.Cu at (138.2, 191.1)
- added TP37: TestPoint, Connector_Pin:Pin_D1.0mm_L10.0mm, F.Cu at (138.2, 195.2)
- added TP38: TestPoint, Connector_Pin:Pin_D1.0mm_L10.0mm, F.Cu at (138.2, 199.2)
- added TP39: TestPoint, Connector_Pin:Pin_D1.0mm_L10.0mm, F.Cu at (142.3, 183.0)
- added TP4: TestPoint, Connector_Pin:Pin_D1.0mm_L10.0mm, F.Cu at (148.3, 201.2)
- added TP40: TestPoint, Connector_Pin:Pin_D1.0mm_L10.0mm, F.Cu at (142.3, 187.1)
- added TP41: TestPoint, Connector_Pin:Pin_D1.0mm_L10.0mm, F.Cu at (142.3, 191.1)
- added TP42: TestPoint, Connector_Pin:Pin_D1.0mm_L10.0mm, F.Cu at (142.3, 195.2)
- added TP43: TestPoint, Connector_Pin:Pin_D1.0mm_L10.0mm, F.Cu at (138.2, 205.3)
- added TP44: TestPoint, Connector_Pin:Pin_D1.0mm_L10.0mm, F.Cu at (138.2, 209.3)
- added TP45: TestPoint, Connector_Pin:Pin_D1.0mm_L10.0mm, F.Cu at (138.2, 213.4)
- added TP46: TestPoint, Connector_Pin:Pin_D1.0mm_L10.0mm, F.Cu at (138.2, 217.4)
- added TP47: TestPoint, Connector_Pin:Pin_D1.0mm_L10.0mm, F.Cu at (142.3, 205.3)
- added TP48: TestPoint, Connector_Pin:Pin_D1.0mm_L10.0mm, F.Cu at (142.3, 209.3)
- added TP49: TestPoint, Connector_Pin:Pin_D1.0mm_L10.0mm, F.Cu at (142.3, 213.4)
- added TP5: TestPoint, Connector_Pin:Pin_D1.0mm_L10.0mm, F.Cu at (148.3, 205.3)
- added TP50: TestPoint, Connector_Pin:Pin_D1.0mm_L10.0mm, F.Cu at (226.1, 152.4)
- added TP51: TestPoint, Connector_Pin:Pin_D1.0mm_L10.0mm, F.Cu at (226.1, 139.7)
- added TP6: TestPoint, Connector_Pin:Pin_D1.0mm_L10.0mm, F.Cu at (148.3, 209.3)
- added TP7: TestPoint, Connector_Pin:Pin_D1.0mm_L10.0mm, F.Cu at (148.3, 213.4)
- added TP8: TestPoint, Connector_Pin:Pin_D1.0mm_L10.0mm, F.Cu at (152.4, 197.2)
- added TP9: TestPoint, Connector_Pin:Pin_D1.0mm_L10.0mm, F.Cu at (152.4, 201.2)
- added U10: 74LS14, Package_DIP:DIP-14_W7.62mm_Socket, F.Cu at (48.3, 25.4)
- added U11: 74LS08, Package_DIP:DIP-14_W7.62mm_Socket, F.Cu at (101.5, 27.9)
- added U12: 74LS02, Package_DIP:DIP-14_W7.62mm_Socket, F.Cu at (114.2, 27.9)
- added U7: L7805, Package_TO_SOT_THT:TO-220-3_Vertical, F.Cu at (25.4, 67.0)
- added U8: L7812/L7815, Package_TO_SOT_THT:TO-220-3_Vertical, F.Cu at (61.0, 172.7)
- C1, C3: value C -> 100nF
- JP1, JP2, JP3, JP4: moved to B.Cu
- T1: value Transformer_1P_1S -> Transformer_1P_2S
- U1, U2: value IR2181 -> IR21814; footprint Package_DIP:DIP-8_W7.62mm_Socket -> Package_DIP:DIP-14_W7.62mm_Socket
- moved R6 281.2 mm to (163.8, 20.3)
- moved R8 273.3 mm to (163.8, 45.7)
- moved U5 262.6 mm to (175.3, -10.2)
- moved U6 251.0 mm to (175.3, 66.0)
- moved Q6 241.7 mm to (447.0, 59.3), turned to 0 degrees
- moved Q5 241.5 mm to (447.0, 53.4), turned to 0 degrees
- moved U4 234.8 mm to (175.3, 40.6)
- moved U3 232.5 mm to (175.3, 15.2)
- moved Q7 224.6 mm to (447.0, 65.3), turned to 0 degrees
- moved Q8 223.5 mm to (447.0, 71.3), turned to 0 degrees
- moved R5 96.5 mm to (426.1, 51.0)
- moved R7 91.6 mm to (426.1, 57.3)
- moved D4 81.0 mm to (239.6, 114.3)
- moved JP7 80.7 mm to (420.7, 69.1)
- moved JP6 80.7 mm to (420.7, 65.5)
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Connections:
- net /Stage_2/ACout_1 renamed /Stage_2/SPWM_1
- net /Stage_2/ACout_2 renamed /Stage_2/SPWM_2
- C1 pad 1: /Stage_1/Vin+ -> VCC
- C3 pad 1: /Stage_1/Vin+ -> VCC
- D1 pad 2: /Stage_1/Vin+ -> Net-(D1-A)
- D2 pad 2: /Stage_1/Vin+ -> Net-(D2-A)
- D3 pad 1: /Stage_2/Vbus+ -> Net-(D3-K)
- D5 pad 1: /Stage_2/Vbus+ -> Net-(D3-K)
- Q1 pad 2: /Stage_1/Vin+ -> Net-(Q1-D)
- Q3 pad 2: /Stage_1/Vin+ -> Net-(Q1-D)
- R6 pad 1: Net-(JP6-A) -> GNDD
- R6 pad 2: Net-(JP6-B) -> Net-(U3-C)
- R7 pad 1: Net-(JP7-A) -> Net-(JP6-A)
- R7 pad 2: Net-(JP7-B) -> Net-(JP6-B)
- R8 pad 1: Net-(JP8-A) -> GNDD
- R8 pad 2: Net-(JP8-B) -> Net-(U4-C)
- T1 pad 1: /Stage_1/Transformer_1 -> Net-(T1-AA)
- T1 pad 2: /Stage_1/Transformer_2 -> Net-(T1-AB)
- T1 pad 3: Net-(D5-A) -> Net-(D3-A)
- T1 pad 4: Net-(D3-A) -> Net-(D5-A)
- U1 pad 1: unconnected-(U1-HIN-Pad1) -> /Control/Stage_1_Gate_2
- U1 pad 2: unconnected-(U1-LIN-Pad2) -> /Control/Stage_1_Gate_1
- U1 pad 3: /Stage_1/Vin- -> GNDD
- U1 pad 4: Net-(JP2-A) -> unconnected-(U1-NC-Pad4)
- U1 pad 5: /Stage_1/Vin+ -> /Stage_1/Vin-
- U1 pad 6: /Stage_1/Transformer_1 -> Net-(JP2-A)
- U1 pad 7: Net-(JP1-A) -> VCC
- U1 pad 8: Net-(D1-K) -> unconnected-(U1-NC-Pad8)
- U2 pad 1: unconnected-(U2-HIN-Pad1) -> /Control/Stage_1_Gate_1
- U2 pad 2: unconnected-(U2-LIN-Pad2) -> /Control/Stage_1_Gate_2
- U2 pad 3: /Stage_1/Vin- -> GNDD
- U2 pad 4: Net-(JP4-A) -> unconnected-(U2-NC-Pad4)
- U2 pad 5: /Stage_1/Vin+ -> /Stage_1/Vin-
- U2 pad 6: /Stage_1/Transformer_2 -> Net-(JP4-A)
- U2 pad 7: Net-(JP3-A) -> VCC
- U2 pad 8: Net-(D2-K) -> unconnected-(U2-NC-Pad8)
- U3 pad 2: unconnected-(U3-A-Pad2) -> /Control/Q5_Gate
- U3 pad 3: unconnected-(U3-C-Pad3) -> Net-(U3-C)
- U3 pad 7: Net-(JP5-A) -> unconnected-(U3-VO-Pad7)
- U3 pad 8: unconnected-(U3-VCC-Pad8) -> /Stage_2/VG_Q5
- U4 pad 2: unconnected-(U4-A-Pad2) -> /Control/Q6_Gate
- U4 pad 3: unconnected-(U4-C-Pad3) -> Net-(U4-C)
- U4 pad 7: Net-(JP6-A) -> unconnected-(U4-VO-Pad7)
- U4 pad 8: unconnected-(U4-VCC-Pad8) -> /Stage_2/VG_Q6_Q8
- U5 pad 2: unconnected-(U5-A-Pad2) -> /Control/Q7_Gate
- U5 pad 3: unconnected-(U5-C-Pad3) -> Net-(U5-C)
- U5 pad 7: Net-(JP7-A) -> unconnected-(U5-VO-Pad7)
- U5 pad 8: unconnected-(U5-VCC-Pad8) -> /Stage_2/VG_Q7
- U6 pad 2: unconnected-(U6-A-Pad2) -> /Control/Q8_Gate
- U6 pad 3: unconnected-(U6-C-Pad3) -> Net-(U6-C)
- U6 pad 7: Net-(JP8-A) -> unconnected-(U6-VO-Pad7)
- U6 pad 8: unconnected-(U6-VCC-Pad8) -> /Stage_2/VG_Q6_Q8
Routing:
- net Net-(JP2-A): track 0.00 -> 27.7 mm
- net Net-(JP4-A): track 0.00 -> 27.1 mm
- net Net-(D1-K): track 0.00 -> 23.9 mm
- net Net-(D2-K): track 0.00 -> 23.9 mm
- net VCC: track 0.00 -> 20.3 mm
- net Net-(JP3-B): track 0.00 -> 16.5 mm
- net Net-(JP1-B): track 0.00 -> 16.5 mm
- net Net-(JP3-A): track 0.00 -> 16.3 mm
- net /Stage_1/Vin-: track 0.00 -> 10.2 mm
- net Net-(D2-A): track 0.00 -> 6.13 mm
- net Net-(D1-A): track 0.00 -> 6.13 mm
- net /Stage_1/Transformer_2: track 0.00 -> 5.11 mm
- net /Stage_1/Transformer_1: track 0.00 -> 5.08 mm
- net Net-(JP4-B): track 0.00 -> 3.78 mm
- net Net-(JP2-B): track 0.00 -> 3.78 mm
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