File: GB2-KiCad/GB2.kicad_sch (KiCad schematic)
At the start: 25 parts, among them J1 Screw_Terminal_01x02, J2 Screw_Terminal_01x02, J3 Barrel_Jack_Switch, J4 Conn_02x10_Odd_Even, T1 Transformer_1P_1S, U7 L7805, U8 L7812/L7815

Commit message: Added shunts and test points
Added shunt resistors and test points to the PCB for debugging purposes.
Parts:
- removed T1: Transformer_1P_1S, GB2:Transformer_GB2_Horizontal, symbol Device:Transformer_1P_1S
- added C38: 400VDC 3.3uF, Capacitor_THT:C_Rect_L33.0mm_W15.0mm_P27.50mm_MKS4, symbol Device:C
- added R22, R23, R24: R_Shunt, Resistor_THT:R_Axial_Shunt_L22.2mm_W8.0mm_PS14.30mm_P25.40mm, symbol Device:R_Shunt
- added T1: Transformer_1P_2S, GB2:Transformer_GB2_Horizontal, symbol Device:Transformer_1P_2S
- added TP1, TP10, TP11, TP12, TP2, TP3, TP4, TP5, TP50, TP51, TP6, TP7, TP8, TP9: TestPoint, Connector_Pin:Pin_D1.0mm_L10.0mm, symbol Connector:TestPoint
- C22, C23, C27, C35: footprint (none) -> Capacitor_THT:CP_Radial_D10.0mm_P2.50mm_P5.00mm
Connections:
- net Stage_1/Transformer_2: now also R22.4
- net Stage_1/Vin+: now also TP1.1
- net Stage_1/Vin-: now also TP2.1
- net Stage_2/SPWM_1: now also TP7.1
- net Stage_2/SPWM_2: now also R24.4; no longer C18.1, J2.2 (Pin_2)
- net Stage_2/Vbus+: now also R23.1; no longer C16.1, L2.2
- net Stage_2/Vbus-: now also C38.1, TP10.1
- net at D3.1 (K), D5.1 (K), L2.1: now also TP9.1
- net at D3.2 (A), D4.1 (K): now also T1.3 (SA)
- net at D5.2 (A), D6.1 (K): now also T1.4 (SB)
- net at C18.2, J2.1 (Pin_1), L3.2: now also TP8.1
- net at C17.2: now also T1.1 (AA)
- new net: R22.1, T1.2 (AB)
- new net: T1.5 (SC), TP51.1
- new net: T1.6 (SD), TP50.1
- new net: C18.1, J2.2 (Pin_2), R24.1
- new net: R24.2, TP6.1
- new net: R24.3, TP5.1
- new net: C16.1, C38.2, L2.2, R23.4
- new net: R23.3, TP11.1
- new net: R23.2, TP12.1
- new net: R22.2, TP4.1
- new net: R22.3, TP3.1
Other:
- moved on the sheet: D4
