File: GB2-KiCad/Stage_1.kicad_sch (KiCad schematic)
At the start: 22 parts, among them Q1 IRF540N, Q2 IRF540N, Q3 IRF540N, Q4 IRF540N, U1 IR21814, U2 IR21814

Commit message: Added shunts and test points
Added shunt resistors and test points to the PCB for debugging purposes.
Parts:
- added R25: R_Shunt, Resistor_THT:R_Axial_Shunt_L22.2mm_W8.0mm_PS14.30mm_P25.40mm, symbol Device:R_Shunt
- added TP29, TP30, TP31, TP32, TP33, TP34, TP35, TP36, TP37, TP38, TP39, TP40, TP41, TP42: TestPoint, Connector_Pin:Pin_D1.0mm_L10.0mm, symbol Connector:TestPoint
Connections:
- net Transformer_1: now also TP31.1
- net Transformer_2: now also TP32.1
- net VCC: now also TP29.1, TP30.1
- net Vin+: now also R25.4; no longer Q1.2 (D), Q3.2 (D)
- net Vin-: now also TP33.1, TP34.1
- net at JP3.2 (B), Q3.1 (G), R3.2: now also TP37.1
- net at C2.1, D1.1 (K), U1.13 (VB): now also TP39.1
- net at JP2.2 (B), Q2.1 (G), R2.2: now also TP36.1
- net at JP4.2 (B), Q4.1 (G), R4.2: now also TP38.1
- net at C4.1, D2.1 (K), U2.13 (VB): now also TP40.1
- net at JP1.2 (B), Q1.1 (G), R1.2: now also TP35.1
- new net: Q1.2 (D), Q3.2 (D), R25.1
- new net: R25.2, TP42.1
- new net: R25.3, TP41.1
