File: GB2-KiCad/Stage_2.kicad_sch (KiCad schematic)
At the start: 47 parts, among them Q5 IPA60R180P7, Q6 IPA60R180P7, Q7 IPA60R180P7, Q8 IPA60R180P7, U3 TLP250, U4 TLP250, U5 TLP250, U6 TLP250

Commit message: Added shunts and test points
Added shunt resistors and test points to the PCB for debugging purposes.
Parts:
- added TP13, TP14, TP15, TP16, TP43, TP44, TP45, TP46, TP47, TP48, TP49: TestPoint, Connector_Pin:Pin_D1.0mm_L10.0mm, symbol Connector:TestPoint
Connections:
- net SPWM_1: now also TP44.1
- net SPWM_2: now also TP45.1
- net VG_Q5: now also TP48.1
- net VG_Q6_Q8: now also TP47.1
- net VG_Q7: now also TP49.1
- net Vbus-: now also TP43.1, TP46.1
- net at JP7.2 (B), Q7.1 (G), R9.2: now also TP15.1
- net at JP8.2 (B), Q8.1 (G), R12.2: now also TP16.1
- net at JP5.2 (B), Q5.1 (G), R5.2: now also TP13.1
- net at JP6.2 (B), Q6.1 (G), R7.2: now also TP14.1
