File: GB2-KiCad/Stage_2.kicad_sch (KiCad schematic)
At the start: 49 parts, among them Q5 IPA60R180P7, Q6 IPA60R180P7, Q7 IPA60R180P7, Q8 IPA60R180P7, U3 TLP250, U4 TLP250, U5 TLP250, U6 TLP250

Commit message: Full pcb layout update
Parts:
- removed R14, R15: R, Resistor_THT:R_Axial_DIN0204_L3.6mm_D1.6mm_P7.62mm_Horizontal, symbol Device:R
Changed lines of the file:
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@@
 	)
 	(junction
-		(at 203.2 31.75)
-		(diameter 0)
-		(color 0 0 0 0)
-	)
-	(junction
 		(at 129.54 31.75)
 		(diameter 0)
@@
 	)
 	(junction
-		(at 203.2 100.33)
-		(diameter 0)
-		(color 0 0 0 0)
-	)
-	(junction
 		(at 72.39 57.15)
 		(diameter 0)
@@
 	(wire
 		(pts
-			(xy 228.6 90.17) (xy 228.6 92.71)
-		)
-		(stroke
-			(width 0)
-			(type default)
-		)
-	)
-	(wire
-		(pts
 			(xy 116.205 57.15) (xy 129.54 57.15)
 		)
@@
 	(wire
 		(pts
-			(xy 203.2 106.68) (xy 203.2 100.33)
+			(xy 203.2 87.63) (xy 203.2 106.68)
 		)
 		(stroke
@@
 	(wire
 		(pts
-			(xy 203.2 31.75) (xy 228.6 31.75)
-		)
-		(stroke
-			(width 0)
-			(type default)
-		)
-	)
-	(wire
-		(pts
 			(xy 139.7 72.39) (xy 152.4 72.39)
 		)
@@
 	(wire
 		(pts
-			(xy 203.2 87.63) (xy 203.2 100.33)
-		)
-		(stroke
-			(width 0)
-			(type default)
-		)
-	)
-	(wire
-		(pts
 			(xy 177.8 72.39) (xy 177.8 80.01)
 		)
@@
 	(wire
 		(pts
-			(xy 228.6 31.75) (xy 228.6 82.55)
-		)
-		(stroke
-			(width 0)
-			(type default)
-		)
-	)
-	(wire
-		(pts
 			(xy 120.65 80.01) (xy 121.92 80.01)
 		)
@@
 	(wire
 		(pts
-			(xy 228.6 100.33) (xy 203.2 100.33)
-		)
-		(stroke
-			(width 0)
-			(type default)
-		)
-	)
-	(wire
-		(pts
 			(xy 115.57 172.72) (xy 119.38 172.72)
 		)
@@
 	)
 	(symbol
-		(lib_id "Device:R")
-		(at 228.6 96.52 180)
-		(unit 1)
-		(exclude_from_sim no)
-		(in_bom yes)
-		(on_board yes)
-		(dnp no)
-		(fields_autoplaced yes)
-		(property "Reference" "R15"
-			(at 231.14 95.2499 0)
-			(effects
-				(font
-					(size 1.27 1.27)
-				)
-				(justify right)
-			)
-		)
-		(property "Value" "R"
-			(at 231.14 97.7899 0)
-			(effects
-				(font
-					(size 1.27 1.27)
-				)
-				(justify right)
-			)
-		)
-		(property "Footprint" "Resistor_THT:R_Axial_DIN0204_L3.6mm_D1.6mm_P7.62mm_Horizontal"
-			(at 230.378 96.52 90)
-			(effects
-				(font
-					(size 1.27 1.27)
-				)
-				(hide yes)
-			)
-		)
-		(property "Datasheet" "~"
-			(at 228.6 96.52 0)
-			(effects
-				(font
-					(size 1.27 1.27)
-				)
-				(hide yes)
-			)
-		)
-		(property "Description" "Resistor"
-			(at 228.6 96.52 0)
-			(effects
-				(font
-					(size 1.27 1.27)
-				)
-				(hide yes)
-			)
-		)
-		(pin "1"
-		)
-		(pin "2"
-		)
-		(instances
-			(project "GB2"
-				(path "/bf64a716-2fc8-4393-9642-a6408cd72f3a/6b5147f6-d1ab-4a6d-b8dc-c38653dffa68"
-					(reference "R15")
-					(unit 1)
-				)
-			)
-		)
-	)
-	(symbol
 		(lib_id "Device:C")
 		(at 177.8 53.34 0)
@@
 					(unit 1)
 				)
-			)
-		)
-	)
-	(symbol
-		(lib_id "Device:R")
-		(at 228.6 86.36 180)
-		(unit 1)
-		(exclude_from_sim no)
-		(in_bom yes)
-		(on_board yes)
-		(dnp no)
-		(fields_autoplaced yes)
-		(property "Reference" "R14"
-			(at 231.14 85.0899 0)
-			(effects
-				(font
-					(size 1.27 1.27)
-				)
-				(justify right)
-			)
-		)
-		(property "Value" "R"
-			(at 231.14 87.6299 0)
-			(effects
-				(font
-					(size 1.27 1.27)
-				)
-				(justify right)
-			)
-		)
-		(property "Footprint" "Resistor_THT:R_Axial_DIN0204_L3.6mm_D1.6mm_P7.62mm_Horizontal"
-			(at 230.378 86.36 90)
-			(effects
-				(font
-					(size 1.27 1.27)
-				)
-				(hide yes)
-			)
-		)
-		(property "Datasheet" "~"
-			(at 228.6 86.36 0)
-			(effects
-				(font
-					(size 1.27 1.27)
-				)
-				(hide yes)
-			)
-		)
-		(property "Description" "Resistor"
-			(at 228.6 86.36 0)
-			(effects
-				(font
-					(size 1.27 1.27)
-				)
-				(hide yes)
-			)
-		)
-		(pin "1"
-		)
-		(pin "2"
-		)
-		(instances
-			(project "GB2"
-				(path "/bf64a716-2fc8-4393-9642-a6408cd72f3a/6b5147f6-d1ab-4a6d-b8dc-c38653dffa68"
-					(reference "R14")
-					(unit 1)
-				)
